File: dlp4710evm-lc-via/LEDBoardBasic.kicad_pcb (KiCad board)
At the start: 2 copper layers, 27.2 x 15.6 mm, 9 parts, among them J1 Molex 874381043

Commit message: dlp4710evm-lc-via_v1 release candidate
Connections:
- net Net-(D1-A) renamed /LED2+
- net Net-(D1-K) renamed /LED-
- net Net-(D3-A) renamed /LED1+
Routing:
- net /LED-: vias 29 -> 51
Other:
- board text added: "DLP4710 EVM-LC- VIA V1"
- board text added: "LED-"
- board text added: "LED1+"
- board text added: "LED2+"
- board text added: "WISHFUL COPPER CORE"
- board text removed: "Anode"
- board text removed: "Cathode"
