File: dlp4710evm-lc-via/LEDBoardBasic.kicad_sch (KiCad schematic)
At the start: 9 parts, among them J1 Molex 874381043

Commit message: dlp4710evm-lc-via_v1 release candidate
Connections:
- net LED-: now reaches D1.1 (K), D2.1 (K), D3.1 (K), D4.1 (K), J1.10_1, J1.10_2, J1.6_1, J1.6_2, J1.7_1, J1.7_2, J1.8_1, J1.8_2, J1.9_1, J1.9_2
- net LED1+: now reaches D3.2 (A), D4.2 (A), J1.1_1, J1.1_2, J1.2_1, J1.2_2
- net LED2+: now reaches D1.2 (A), D2.2 (A), J1.3_1, J1.3_2, J1.4_1, J1.4_2, J1.5_1, J1.5_2
Changed lines of the file:
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@@
+		)
+	)
+	(label "LED1+"
+		(at 156.21 116.84 90)
+		(effects
+			(font
+				(size 1.27 1.27)
+			)
+			(justify left bottom)
+		)
+	)
+	(label "LED-"
+		(at 133.35 71.12 180)
+		(effects
+			(font
+				(size 1.27 1.27)
+			)
+			(justify right bottom)
+		)
+	)
+	(label "LED2+"
+		(at 152.4 100.33 90)
+		(effects
+			(font
+				(size 1.27 1.27)
+			)
+			(justify left bottom)
 		)
 	)

Commit message: Added footprints
Added mechanical hole footprints which were missing from project library.
Parts:
- H1, H2: footprint LaughingsSynthFootprints:0dot093_inch_mechanical_hole -> LEDBoardLibrary:0dot093_inch_mechanical_hole
- H3, H4: footprint LaughingsSynthFootprints:0dot060_inch_mechanical_hole -> LEDBoardLibrary:0dot060_inch_mechanical_hole
Changed lines of the file:
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@@
 			)
 		)
-		(property "Footprint" "LaughingsSynthFootprints:0dot093_inch_mechanical_hole"
+		(property "Footprint" "LEDBoardLibrary:0dot093_inch_mechanical_hole"
 			(at 109.22 102.87 0)
 			(effects
@@
 			)
 		)
-		(property "Footprint" "LaughingsSynthFootprints:0dot093_inch_mechanical_hole"
+		(property "Footprint" "LEDBoardLibrary:0dot093_inch_mechanical_hole"
 			(at 109.22 96.52 0)
 			(effects
@@
 			)
 		)
-		(property "Footprint" "LaughingsSynthFootprints:0dot060_inch_mechanical_hole"
+		(property "Footprint" "LEDBoardLibrary:0dot060_inch_mechanical_hole"
 			(at 88.9 96.52 0)
 			(effects
@@
 			)
 		)
-		(property "Footprint" "LaughingsSynthFootprints:0dot060_inch_mechanical_hole"
+		(property "Footprint" "LEDBoardLibrary:0dot060_inch_mechanical_hole"
 			(at 88.9 102.87 0)
 			(effects
